File: kp_ledsuit.kicad_pcb (KiCad board)
At the start: 2 copper layers, 63.1 x 36.5 mm, 79 parts, among them IC1 MP2359DJ-LF-Z, J1 USB_B_Mini, J2 SWD, J3 Conn_01x04_MountingPin, J4 SK9822, Q1 AO3401A, Q2 BC818, SW1 SW_SPDT, U1 STM32F103C8Tx, U2 USBLC6-2P6, U3 LSM6DS3, Y1 12MHz

Commit message: WIP first proto layout: 1 face
Parts:
- C1, C10, C11, C13, C14, C15, C19, C2, C22, C3, C5, C6, C8, D2, D4, D7, F1, FB1, FB2, IC1, L1, Q1, Q2, R1, R10, R11, R19, R24, R25, R26, R3, R5, R9, U3: moved to F.Cu
- moved H1 102.7 mm to (122.0, 123.0)
- moved R14 69.7 mm to (139.0, 118.0), turned to 180 degrees
- moved C17 68.9 mm to (130.8, 112.0), turned to -90 degrees
- moved C16 67.0 mm to (133.2, 112.0), turned to -90 degrees
- moved R15 66.4 mm to (128.6, 85.6), turned to -90 degrees
- moved R16 63.9 mm to (129.9, 85.6), turned to -90 degrees
- moved L1 63.7 mm to (137.9, 111.2)
- moved R13 63.2 mm to (143.7, 118.0), turned to 180 degrees
- moved R17 61.4 mm to (131.2, 85.6), turned to -90 degrees
- moved J2 60.8 mm to (131.2, 81.1), turned to 90 degrees
- moved R12 60.0 mm to (143.8, 115.6), turned to 0 degrees
- moved R23 59.0 mm to (133.8, 119.5)
- moved R22 59.0 mm to (132.5, 119.5)
- moved J3 59.0 mm to (133.1, 124.4)
- moved FB2 58.4 mm to (148.2, 110.5), turned to 180 degrees
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Routing:
- added copper zone on In1.Cu, net +3.3V
- added copper zone on B.Cu, net GND
- added copper zone on F.Cu, net GND
- added copper zone on In2.Cu, net GND
Other:
- board size 63.1 x 36.5 mm -> 50 x 50 mm
- copper layers 2 -> 4

Commit message: pxm test logo
Parts:
- added G***: LOGO, homemade_footprints:pxm_testlogo_v1, F.Cu at (154.8, 121.8)
- moved C13 0.20 mm to (142.0, 111.2)
- moved C12 0.10 mm to (128.0, 95.2)
- moved R7 0.09 mm to (129.5, 94.8)
- moved C7 0.06 mm to (145.8, 79.8)
- moved C10 0.06 mm to (165.3, 97.6)
Other:
- board text added: "ledsuit_00"

Commit message: WIP
Parts:
- removed C10, C18, C19, C20, C21, C7, C8, C9: 100n, Capacitor_SMD:C_0402_1005Metric
- C2: footprint Capacitor_SMD:C_0805_2012Metric -> Capacitor_SMD:C_1206_3216Metric
- D1, D3, D6: value Y/W/G -> G
- D2, D4, D7: value Y/W/G -> Y
- D8, D9: value Y/W/G -> W
- R10, R11: value TODO -> 400
- R2, R4, R8: value TODO -> 450
- R3, R5, R9: value TODO -> 1200
- R7: value 47 -> 33
- moved D6 5.60 mm to (159.3, 116.7)
- moved R8 5.60 mm to (161.3, 116.7)
- moved R9 4.03 mm to (155.1, 114.7)
- moved D7 4.00 mm to (157.1, 114.8)
- moved D1 1.13 mm to (144.6, 78.7)
- moved R2 1.13 mm to (144.5, 80.7)
- moved C5 0.21 mm to (136.2, 90.3)
- moved R11 0.08 mm to (162.2, 86.8), turned to 180 degrees
- moved C2 0.06 mm to (147.1, 92.3)
Routing:
- net +3.3V: track 0.00 -> 74.5 mm, vias 0 -> 30
- net TIM2_CH1: track 0.00 -> 61.3 mm, vias 0 -> 2
- net TIM4_CH2: track 0.00 -> 53.6 mm, vias 0 -> 2
- net USB_CONN_5V: track 0.00 -> 51.2 mm, vias 0 -> 6
- net GND: track 0.00 -> 51.0 mm, vias 0 -> 14
- net TIM2_CH2: track 0.00 -> 47.8 mm, vias 0 -> 2
- net TIM2_CH4: track 0.00 -> 41.2 mm, vias 0 -> 2
- net SPI2_SCK: track 0.00 -> 40.1 mm, vias 0 -> 2
- net SPI2_MOSI: track 0.00 -> 39.0 mm, vias 0 -> 2
- net TIM4_CH4: track 0.00 -> 38.9 mm, vias 0 -> 2
- net TIM2_CH3: track 0.00 -> 36.2 mm, vias 0 -> 2
- net USART1_RX: track 0.00 -> 28.4 mm, vias 0 -> 2
- net USART1_TX: track 0.00 -> 27.6 mm, vias 0 -> 2
- net TIM4_CH3: track 0.00 -> 23.4 mm, vias 0 -> 2
- net BUCK_EN: track 0.00 -> 23.2 mm, vias 0 -> 2
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- added copper zone on In2.Cu, net +3.3V
- added copper zone on In1.Cu, net GND
- added copper zone on In2.Cu, net USB_CONN_5V
- removed copper zone on In1.Cu, net +3.3V
- removed copper zone on In2.Cu, net GND

Commit message: v00 - send to prod
Parts:
- added H5: tooling, homemade_footprints:jlc_tooling_hole, F.Cu at (125.9, 79.1)
- added H6: tooling, homemade_footprints:jlc_tooling_hole, F.Cu at (125.7, 124.7)
- added H7: tooling, homemade_footprints:jlc_tooling_hole, F.Cu at (160.7, 78.6)
- R10, R11: value 400 -> 470
- R2, R4, R8: value 450 -> 470
- R3, R5, R9: value 1200 -> 1.02k
- moved D2 0.25 mm to (144.7, 125.5)
- moved R3 0.25 mm to (144.8, 123.5)
Routing:
- net +3.3V: track 74.5 -> 75.0 mm
- net GND: vias 14 -> 42
