File: kp_ledsuit.kicad_sch (KiCad schematic)
At the start: 79 parts, among them IC1 MP2359DJ-LF-Z, J1 USB_B_Mini, J2 SWD, J3 Conn_01x04_MountingPin, J4 SK9822, Q1 AO3401A, Q2 BC818, SW1 SW_SPDT, U1 STM32F103C8Tx, U2 USBLC6-2P6, U3 LSM6DS3, Y1 12MHz

Commit message: WIP
Parts:
- removed C10, C18, C19, C20, C21, C7, C8, C9: 100n, Capacitor_SMD:C_0402_1005Metric, symbol Device:C_Small
- C1, C16, C17: JLCPCB Part # (none) -> C13585
- C11, C15, C22, C23, C24, C3, C5, C6: JLCPCB Part # (none) -> C307331
- C12, C4: JLCPCB Part # (none) -> C1554
- C13: JLCPCB Part # (none) -> C57112
- C14: JLCPCB Part # (none) -> C28323
- C2: footprint Capacitor_SMD:C_0805_2012Metric -> Capacitor_SMD:C_1206_3216Metric; JLCPCB Part # (none) -> C13585
- D1, D3, D6: value Y/W/G -> G
- D2, D4, D7: value Y/W/G -> Y; JLCPCB Part # C2297 -> C2296
- D8, D9: value Y/W/G -> W; JLCPCB Part # C2297 -> C34499
- Q2: JLCPCB Part # (none) -> C154797
- R1, R20, R25, R26, R6: JLCPCB Part # (none) -> C25804
- R10, R11: value TODO -> 400
- R15, R16, R17, R18, R22, R23: JLCPCB Part # (none) -> C25092
- R19: JLCPCB Part # (none) -> C22775
- R2, R4, R8: value TODO -> 450
- R24: JLCPCB Part # (none) -> C22843
- R3, R5, R9: value TODO -> 1200
- R7: value 47 -> 33; JLCPCB Part # (none) -> C25105

Commit message: v00 - send to prod
Parts:
- added H5, H6, H7: tooling, homemade_footprints:jlc_tooling_hole, symbol Mechanical:MountingHole
- R10, R11: value 400 -> 470; JLCPCB Part # (none) -> C17710
- R2, R4, R8: value 450 -> 470; JLCPCB Part # (none) -> C17710
- R20: JLCPCB Part # C25804 -> (none)
- R3, R5, R9: value 1200 -> 1.02k; JLCPCB Part # (none) -> C17369
Other:
- note added: "jlc tooling holes"
Changed lines of the file:
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@@
     (stroke (width 0) (type default))
   )
+  (polyline (pts (xy 384.81 57.15) (xy 384.81 86.36))
+    (stroke (width 0) (type dot))
+  )
   (wire (pts (xy 53.34 158.75) (xy 53.34 160.02))
     (stroke (width 0) (type default))
@@
     (stroke (width 0) (type default))
   )
+  (polyline (pts (xy 361.95 57.15) (xy 361.95 86.36))
+    (stroke (width 0) (type dot))
+  )
   (wire (pts (xy 143.51 120.65) (xy 148.59 120.65))
     (stroke (width 0) (type default))
@@
     (stroke (width 0) (type default))
   )
+  (polyline (pts (xy 384.81 86.36) (xy 361.95 86.36))
+    (stroke (width 0) (type dot))
+  )
   (wire (pts (xy 93.98 57.15) (xy 93.98 63.5))
     (stroke (width 0) (type default))
@@
     (stroke (width 0) (type dot))
   )
+  (polyline (pts (xy 361.95 57.15) (xy 384.81 57.15))
+    (stroke (width 0) (type dot))
+  )
   (wire (pts (xy 86.36 124.46) (xy 88.9 124.46))
     (stroke (width 0) (type default))
@@
     (effects (font (size 1.27 1.27)) (justify left bottom))
   )
+  (text "jlc tooling holes" (at 365.76 60.96 0)
+    (effects (font (size 1.27 1.27)) (justify left bottom))
+  )
   (text "output regulating" (at 87.63 54.61 0)
     (effects (font (size 1.27 1.27)) (justify left bottom))
@@
     )
   )
+  (symbol (lib_id "Mechanical:MountingHole") (at 369.57 81.28 0) (unit 1)
+    (in_bom yes) (on_board yes) (dnp no) (fields_autoplaced)
+    (property "Reference" "H7" (at 372.11 80.01 0)
+      (effects (font (size 1.27 1.27)) (justify left))
+    )
+    (property "Value" "tooling" (at 372.11 82.55 0)
+      (effects (font (size 1.27 1.27)) (justify left))
+    )
+    (property "Footprint" "homemade_footprints:jlc_tooling_hole" (at 369.57 81.28 0)
+      (effects (font (size 1.27 1.27)) hide)
+    )
+    (property "Datasheet" "~" (at 369.57 81.28 0)
+      (effects (font (size 1.27 1.27)) hide)
+    )
+    (instances
+      (project "kp_ledsuit"
+        (path "/79a1ace3-82e7-4ba1-acff-a1e56b662ec8"
+          (reference "H7") (unit 1)
+        )
+      )
+    )
+  )
   (symbol (lib_id "power:GND") (at 110.49 163.83 0) (unit 1)
     (in_bom yes) (on_board yes) (dnp no)
@@
       (effects (font (size 1.27 1.27)))
     )
-    (property "Value" "1200" (at 35.56 109.22 90)
+    (property "Value" "1.02k" (at 35.56 109.22 90)
       (effects (font (size 1.27 1.27)))
     )
@@
       (effects (font (size 1.27 1.27)) hide)
     )
-    (property "JLCPCB Part #" "" (at 35.56 106.68 0)
+    (property "JLCPCB Part #" "C17369" (at 35.56 106.68 0)
       (effects (font (size 1.27 1.27)) hide)
     )
@@
       (effects (font (size 1.27 1.27)))
     )
-    (property "Value" "450" (at 83.82 100.33 90)
+    (property "Value" "470" (at 83.82 100.33 90)
       (effects (font (size 1.27 1.27)))
     )
@@
       (effects (font (size 1.27 1.27)) hide)
     )
-    (property "JLCPCB Part #" "" (at 83.82 97.79 0)
+    (property "JLCPCB Part #" "C17710" (at 83.82 97.79 0)
       (effects (font (size 1.27 1.27)) hide)
     )
@@
       (effects (font (size 1.27 1.27)))
     )
-    (property "Value" "450" (at 35.56 100.33 90)
+    (property "Value" "470" (at 35.56 100.33 90)
       (effects (font (size 1.27 1.27)))
     )
@@
       (effects (font (size 1.27 1.27)) hide)
     )
-    (property "JLCPCB Part #" "" (at 35.56 97.79 0)
+    (property "JLCPCB Part #" "C17710" (at 35.56 97.79 0)
       (effects (font (size 1.27 1.27)) hide)
     )
@@
       (effects (font (size 1.27 1.27)))
     )
-    (property "Value" "400" (at 83.82 127 90)
+    (property "Value" "470" (at 83.82 127 90)
       (effects (font (size 1.27 1.27)))
     )
@@
       (effects (font (size 1.27 1.27)) hide)
     )
-    (property "JLCPCB Part #" "" (at 83.82 124.46 0)
+    (property "JLCPCB Part #" "C17710" (at 83.82 124.46 0)
       (effects (font (size 1.27 1.27)) hide)
     )
@@
       (effects (font (size 1.27 1.27)))
     )
-    (property "Value" "450" (at 35.56 118.11 90)
+    (property "Value" "470" (at 35.56 118.11 90)
       (effects (font (size 1.27 1.27)))
     )
@@
       (effects (font (size 1.27 1.27)) hide)
     )
-    (property "JLCPCB Part #" "" (at 35.56 115.57 0)
+    (property "JLCPCB Part #" "C17710" (at 35.56 115.57 0)
       (effects (font (size 1.27 1.27)) hide)
     )
@@
     )
   )
+  (symbol (lib_id "Mechanical:MountingHole") (at 369.57 66.04 0) (unit 1)
+    (in_bom yes) (on_board yes) (dnp no) (fields_autoplaced)
+    (property "Reference" "H5" (at 372.11 64.77 0)
+      (effects (font (size 1.27 1.27)) (justify left))
+    )
+    (property "Value" "tooling" (at 372.11 67.31 0)
+      (effects (font (size 1.27 1.27)) (justify left))
+    )
+    (property "Footprint" "homemade_footprints:jlc_tooling_hole" (at 369.57 66.04 0)
+      (effects (font (size 1.27 1.27)) hide)
+    )
+    (property "Datasheet" "~" (at 369.57 66.04 0)
+      (effects (font (size 1.27 1.27)) hide)
+    )
+    (instances
+      (project "kp_ledsuit"
+        (path "/79a1ace3-82e7-4ba1-acff-a1e56b662ec8"
+          (reference "H5") (unit 1)
+        )
+      )
+    )
+  )
   (symbol (lib_id "power:+3.3V") (at 48.26 92.71 0) (unit 1)
     (in_bom yes) (on_board yes) (dnp no)
@@
       (effects (font (size 1.27 1.27)))
     )
-    (property "Value" "400" (at 83.82 118.11 90)
+    (property "Value" "470" (at 83.82 118.11 90)
       (effects (font (size 1.27 1.27)))
     )
@@
       (effects (font (size 1.27 1.27)) hide)
     )
-    (property "JLCPCB Part #" "" (at 83.82 115.57 0)
+    (property "JLCPCB Part #" "C17710" (at 83.82 115.57 0)
       (effects (font (size 1.27 1.27)) hide)
     )
@@
       (effects (font (size 1.27 1.27)))
     )
-    (property "Value" "1200" (at 35.56 127 90)
+    (property "Value" "1.02k" (at 35.56 127 90)
       (effects (font (size 1.27 1.27)))
     )
@@
       (effects (font (size 1.27 1.27)) hide)
     )
-    (property "JLCPCB Part #" "" (at 35.56 124.46 0)
+    (property "JLCPCB Part #" "C17369" (at 35.56 124.46 0)
       (effects (font (size 1.27 1.27)) hide)
     )
@@
       (effects (font (size 1.27 1.27)) hide)
     )
-    (property "JLCPCB Part #" "C25804" (at 181.61 170.18 0)
+    (property "JLCPCB Part #" "" (at 181.61 170.18 0)
       (effects (font (size 1.27 1.27)) hide)
     )
@@
     )
   )
+  (symbol (lib_id "Mechanical:MountingHole") (at 369.57 73.66 0) (unit 1)
+    (in_bom yes) (on_board yes) (dnp no) (fields_autoplaced)
+    (property "Reference" "H6" (at 372.11 72.39 0)
+      (effects (font (size 1.27 1.27)) (justify left))
+    )
+    (property "Value" "tooling" (at 372.11 74.93 0)
+      (effects (font (size 1.27 1.27)) (justify left))
+    )
+    (property "Footprint" "homemade_footprints:jlc_tooling_hole" (at 369.57 73.66 0)
+      (effects (font (size 1.27 1.27)) hide)
+    )
+    (property "Datasheet" "~" (at 369.57 73.66 0)
+      (effects (font (size 1.27 1.27)) hide)
+    )
+    (instances
+      (project "kp_ledsuit"
+        (path "/79a1ace3-82e7-4ba1-acff-a1e56b662ec8"
+          (reference "H6") (unit 1)
+        )
+      )
+    )
+  )
   (symbol (lib_id "Connector_Generic:Conn_02x05_Odd_Even") (at 135.89 120.65 0) (unit 1)
     (in_bom yes) (on_board yes) (dnp no)
@@
       (effects (font (size 1.27 1.27)))
     )
-    (property "Value" "1200" (at 83.82 109.22 90)
+    (property "Value" "1.02k" (at 83.82 109.22 90)
       (effects (font (size 1.27 1.27)))
     )
@@
       (effects (font (size 1.27 1.27)) hide)
     )
-    (property "JLCPCB Part #" "" (at 83.82 106.68 0)
+    (property "JLCPCB Part #" "C17369" (at 83.82 106.68 0)
       (effects (font (size 1.27 1.27)) hide)
     )
